Commit message: feat(g1): add minimal reproducible MoveIt XR deployment

File: ros2_ws/src/g1_description/urdf/g1_29dof_with_inspire_hand_ftp.urdf (robot description, URDF)
Before this commit: robot g1_29dof_rev_1_0_with_inspire_hand_FTP, 97 links, 96 joints
Links:
- link pelvis: geometry collision mesh filename=package://g1_description/meshes/pelvis.STL; visual mesh filename=package://g1_description/meshes/pelvis.STL
- link waist_roll_link: geometry collision mesh filename=package://g1_description/meshes/waist_roll_link_rev_1_0.STL; visual mesh filename=package://g1_description/meshes/waist_roll_link_rev_1_0.STL
- link waist_yaw_link: geometry collision mesh filename=package://g1_description/meshes/waist_yaw_link_rev_1_0.STL; visual mesh filename=package://g1_description/meshes/waist_yaw_link_rev_1_0.STL
